Commit message: Rename Solidworks export

File: src/sparky_description/urdf/sparky_description.urdf (robot description, URDF)
Before this commit: robot MR24-DT-A00.00_URDF, 7 links, 6 joints
Links:
- link Center_Left Wheel: geometry collision mesh filename=package://sparky_description/meshes/Center_Left Wheel.STL; visual mesh filename=package://sparky_description/meshes/Center_Left Wheel.STL
- link Center_Right Wheel: geometry collision mesh filename=package://sparky_description/meshes/Center_Right Wheel.STL; visual mesh filename=package://sparky_description/meshes/Center_Right Wheel.STL
- link Front_Left Wheel: geometry collision mesh filename=package://sparky_description/meshes/Front_Left Wheel.STL; visual mesh filename=package://sparky_description/meshes/Front_Left Wheel.STL
- link Front_right Wheel: geometry collision mesh filename=package://sparky_description/meshes/Front_right Wheel.STL; visual mesh filename=package://sparky_description/meshes/Front_right Wheel.STL
- link Rear_Left Wheel: geometry collision mesh filename=package://sparky_description/meshes/Rear_Left Wheel.STL; visual mesh filename=package://sparky_description/meshes/Rear_Left Wheel.STL
- link Rear_Right Wheel: geometry collision mesh filename=package://sparky_description/meshes/Rear_Right Wheel.STL; visual mesh filename=package://sparky_description/meshes/Rear_Right Wheel.STL
- link base_link: geometry collision mesh filename=package://sparky_description/meshes/base_link.STL; visual mesh filename=package://sparky_description/meshes/base_link.STL

Commit message: noetic urdf rviz validated

File: src/sparky_description/urdf/sparky_description.urdf (robot description, URDF)
Before this commit: robot sparky_description, 7 links, 6 joints
Links:
- removed link Center_Left Wheel
- removed link Center_Right Wheel
- removed link Front_Left Wheel
- removed link Front_right Wheel
- removed link Rear_Left Wheel
- removed link Rear_Right Wheel
- added link Center_Left_Wheel, mass 1.45375895562015; collision mesh filename=package://sparky_description/meshes/Center_Left_Wheel.STL; visual mesh filename=package://sparky_description/meshes/Center_Left_Wheel.STL
- added link Center_Right_Wheel, mass 1.45375895562016; collision mesh filename=package://sparky_description/meshes/Center_Right_Wheel.STL; visual mesh filename=package://sparky_description/meshes/Center_Right_Wheel.STL
- added link Front_Left_Wheel, mass 1.45375895562109; collision mesh filename=package://sparky_description/meshes/Front_Left_Wheel.STL; visual mesh filename=package://sparky_description/meshes/Front_Left_Wheel.STL
- added link Front_right_Wheel, mass 1.45375895562017; collision mesh filename=package://sparky_description/meshes/Front_right_Wheel.STL; visual mesh filename=package://sparky_description/meshes/Front_right_Wheel.STL
- added link Rear_Left_Wheel, mass 1.45375895562016; collision mesh filename=package://sparky_description/meshes/Rear_Left_Wheel.STL; visual mesh filename=package://sparky_description/meshes/Rear_Left_Wheel.STL
- added link Rear_Right_Wheel, mass 1.45375895562016; collision mesh filename=package://sparky_description/meshes/Rear_Right_Wheel.STL; visual mesh filename=package://sparky_description/meshes/Rear_Right_Wheel.STL
Joints:
- removed joint Center_Left Wheel Joint
- removed joint Center_Right Wheel Joint
- removed joint Front_Left Wheel Joint
- removed joint Front_Right Wheel Joint
- removed joint Rear_Left Wheel Joint
- removed joint Rear_Right Wheel Joint
- added joint Center_Left_Wheel_Joint: type continuous, parent base_link, child Center_Left_Wheel, origin xyz=0 0.48455 0 rpy=1.5708 0 0, axis 0 0 1
- added joint Center_Right_Wheel_Joint: type continuous, parent base_link, child Center_Right_Wheel, origin xyz=0 -0.48455 0 rpy=1.5708 0 0, axis 0 0 -1
- added joint Front_Left_Wheel_Joint: type continuous, parent base_link, child Front_Left_Wheel, origin xyz=0.40398 0.43855 0.0080468 rpy=1.5708 0 0, axis 0 0 1
- added joint Front_Right_Wheel_Joint: type continuous, parent base_link, child Front_right_Wheel, origin xyz=0.40398 -0.43855 0.0080468 rpy=1.5708 0 0, axis 0 0 -1
- added joint Rear_Left_Wheel_Joint: type continuous, parent base_link, child Rear_Left_Wheel, origin xyz=-0.39807 0.48455 0.016315 rpy=1.5708 0 0, axis 0 0 1
- added joint Rear_Right_Wheel_Joint: type continuous, parent base_link, child Rear_Right_Wheel, origin xyz=-0.39807 -0.48455 0.016315 rpy=1.5708 0 0, axis 0 0 -1
