Commit message: update kinematics fix

File: src/sparky_description/urdf/sparky.ros2_control.xacro (robot description, xacro)
@@ -20,8 +20,12 @@
       </xacro:unless>
       <!-- Per-wheel joint definition. node_id is only used by the ODrive
-           backend; mock_components ignores it. -->
-      <xacro:macro name="drive_joint" params="name node_id">
+           backend; mock_components ignores it. direction (+1/-1) is the sign the
+           ODrive backend applies to commands and feedback: the left wheels are
+           mirror-mounted, so they get -1 to spin the correct way for forward
+           motion. mock_components ignores direction too. -->
+      <xacro:macro name="drive_joint" params="name node_id direction:=1">
         <joint name="${name}">
           <param name="node_id">${node_id}</param>
+          <param name="direction">${direction}</param>
           <command_interface name="velocity"/>
           <state_interface name="position"/>
@@ -30,8 +34,8 @@
         </joint>
       </xacro:macro>
-      <!-- Left side -->
-      <xacro:drive_joint name="Front_Left_Wheel_Joint"  node_id="4"/>
-      <xacro:drive_joint name="Center_Left_Wheel_Joint" node_id="5"/>
-      <xacro:drive_joint name="Rear_Left_Wheel_Joint"   node_id="6"/>
+      <!-- Left side (mirror-mounted: inverted) -->
+      <xacro:drive_joint name="Front_Left_Wheel_Joint"  node_id="4" direction="-1"/>
+      <xacro:drive_joint name="Center_Left_Wheel_Joint" node_id="5" direction="-1"/>
+      <xacro:drive_joint name="Rear_Left_Wheel_Joint"   node_id="6" direction="-1"/>
       <!-- Right side -->
       <xacro:drive_joint name="Front_Right_Wheel_Joint"  node_id="1"/>
