Commit message: Refactor sparky_description and consolidate bringup launch/config files
Splits drivetrain/groundstation launch files apart from sparky_description,
moves rviz configs and stray scripts into their owning packages, and cleans
up package.xml/CMakeLists dependencies to match.

Co-Authored-By: Claude Sonnet 5 <noreply@anthropic.com>

File: src/sparky_description/urdf/sparky.control.urdf.xacro (robot description, xacro)
@@ -1,10 +1,9 @@
 <?xml version="1.0"?>
 <!--
-  ros2_control on UWRobotics Sparky URDF.
+  UWRobotics Sparky URDF Package
 -->
 <robot xmlns:xacro="http://www.ros.org/wiki/xacro" name="sparky">
-  <!-- Testing with Software Components Only -->
+  <!-- Launch File Pass-in Args -->
   <xacro:arg name="use_mock_hardware" default="true"/>
-  <!-- Launch with Can Instance Default match Jetson -->
   <xacro:arg name="can_interface"     default="can2"/>
   <xacro:include filename="$(find sparky_description)/urdf/sparky_description.urdf"/>

File: src/sparky_description/urdf/sparky.ros2_control.xacro (robot description, xacro)
@@ -2,30 +2,23 @@
 <robot xmlns:xacro="http://www.ros.org/wiki/xacro">
   <!--
-    ros2_control hardware description for the Sparky CIRC 2026 rover.
+    UWRobotics Sparky ros2_control package
   -->
-  <xacro:macro name="sparky_ros2_control"
-               params="name use_mock_hardware:=true can_interface:=can0">
+  <xacro:macro name="sparky_ros2_control" params="name use_mock_hardware can_interface">
     <ros2_control name="${name}" type="system">
-      <xacro:if value="${use_mock_hardware}">
-        <hardware>
+      <hardware>
+        <xacro:if value="${use_mock_hardware}">
           <plugin>mock_components/GenericSystem</plugin>
           <param name="calculate_dynamics">true</param>
-        </hardware>
-      </xacro:if>
-      <xacro:unless value="${use_mock_hardware}">
-        <hardware>
+        </xacro:if>
+        <xacro:unless value="${use_mock_hardware}">
           <plugin>odrive_ros2_control_plugin/ODriveHardwareInterface</plugin>
           <param name="can">${can_interface}</param>
-        </hardware>
-      </xacro:unless>
-      <!-- Per-wheel joint definition. node_id is only used by the ODrive
-           backend; mock_components ignores it. direction (+1/-1) is the sign the
-           ODrive backend applies to commands and feedback: the left wheels are
-           mirror-mounted, so they get -1 to spin the correct way for forward
-           motion. mock_components ignores direction too. -->
-      <xacro:macro name="drive_joint" params="name node_id direction:=1">
+        </xacro:unless>
+      </hardware>
+      <xacro:macro name="drive_joint" params="name node_id direction:=1 gear_ratio:=35">
         <joint name="${name}">
           <param name="node_id">${node_id}</param>
           <param name="direction">${direction}</param>
+          <param name="gear_ratio">${gear_ratio}</param>
           <command_interface name="velocity"/>
           <state_interface name="position"/>
@@ -34,5 +27,5 @@
         </joint>
       </xacro:macro>
-      <!-- Left side (mirror-mounted: inverted) -->
+      <!-- Left side (inverted) -->
       <xacro:drive_joint name="Front_Left_Wheel_Joint"  node_id="4" direction="-1"/>
       <xacro:drive_joint name="Center_Left_Wheel_Joint" node_id="5" direction="-1"/>
