Commit message: ros2 support change

File: src/arm_description/urdf/dummy_urdf.urdf (robot description, URDF)
Before this commit: robot dummy_urdf, 7 links, 6 joints
Links:
- link Gripper: geometry collision mesh filename=package://arm_description/meshes/Gripper.STL; visual mesh filename=package://arm_description/meshes/Gripper.STL
- link Link_1: geometry collision mesh filename=package://arm_description/meshes/Link_1.STL; visual mesh filename=package://arm_description/meshes/Link_1.STL
- link Link_2: geometry collision mesh filename=package://arm_description/meshes/Link_2.STL; visual mesh filename=package://arm_description/meshes/Link_2.STL
- link Link_3: geometry collision mesh filename=package://arm_description/meshes/Link_3.STL; visual mesh filename=package://arm_description/meshes/Link_3.STL
- link Link_4: geometry collision mesh filename=package://arm_description/meshes/Link_4.STL; visual mesh filename=package://arm_description/meshes/Link_4.STL
- link Link_5: geometry collision mesh filename=package://arm_description/meshes/Link_5.STL; visual mesh filename=package://arm_description/meshes/Link_5.STL
- link Link_6: geometry collision mesh filename=package://arm_description/meshes/Link_6.STL; visual mesh filename=package://arm_description/meshes/Link_6.STL
