Commit message: add joint limits to URDF and new arm_moveit_config package

File: src/arm_description/urdf/dummy_urdf.urdf (robot description, URDF)
Before this commit: robot dummy_urdf, 7 links, 6 joints
Joints:
- joint Joint_1: limit (none) -> effort=0 velocity=5.236
- joint Joint_2: limit (none) -> lower=0.0349 upper=3.1765 effort=0 velocity=0.873; type continuous -> revolute
- joint Joint_3: limit (none) -> lower=0.0349 upper=3.1765 effort=0 velocity=1.080; type continuous -> revolute
- joint Joint_4: limit (none) -> effort=0 velocity=1.007
- joint Joint_5: limit (none) -> lower=-0.9774 upper=1.8850 effort=0 velocity=1.007; type continuous -> revolute
- joint Joint_6: limit (none) -> effort=0 velocity=1.007
